File: hardware/temperature-sensor/fan.kicad_sch (KiCad schematic)
At the start: 0 parts

Commit message: work on temperature sensor
Parts:
- added D8: BAT54WS, benediktibk:D_SOD-323, symbol benediktibk:BAT54WS
- added J3: 1990012, benediktibk:1990012, symbol benediktibk:1990012
- added Q1: DMN3404L, benediktibk:SOT-23, symbol benediktibk:DMN3404L
- added R26, R27: 10kOhm, benediktibk:R_0603_1608Metric_Pad0.98x0.95mm_HandSolder, symbol benediktibk:R_10kOhm_SMD_0603_100mW_1%
Connections:
- new net: D8.2 (A), J3.3, Q1.3 (D)
- new net 12V: D8.1 (K), J3.1
- new net 3V3: R26.1
- new net GND: Q1.2 (S), R27.2
- new net PWM: Q1.1 (G), R27.1
- new net TACH: J3.2, R26.2
Other:
- note added: "Selected Fan: 472-04010SS-12N-AT00 3 wire (one Tach signal) 12VDC 710mW"
