File: hardware/temperature-sensor/Ethernet.kicad_sch (KiCad schematic)
At the start: 27 parts, among them J1 1149611, T1 SM13126PEL, U2 LAN8720A

Commit message: update symbols from library
Parts:
- R5, R6, R7, R8: Mouser Part Number (none) -> 603-AC0603FR-1347RL
Changed lines of the file:
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@@
+			)
+		)
+		(property "Mouser Part Number" "603-AC0603FR-1347RL"
+			(at 129.54 52.07 0)
+			(effects
+				(font
+					(size 1.27 1.27)
+				)
+				(hide yes)
 			)
 		)
@@
 			)
 		)
+		(property "Mouser Part Number" "603-AC0603FR-1347RL"
+			(at 95.25 52.07 0)
+			(effects
+				(font
+					(size 1.27 1.27)
+				)
+				(hide yes)
+			)
+		)
 		(pin "2"
 		)
@@
 			)
 		)
+		(property "Mouser Part Number" "603-AC0603FR-1347RL"
+			(at 106.68 52.07 0)
+			(effects
+				(font
+					(size 1.27 1.27)
+				)
+				(hide yes)
+			)
+		)
 		(pin "2"
 		)
@@
 			(effects
 				(font
+					(size 1.27 1.27)
+				)
+				(hide yes)
+			)
+		)
+		(property "Mouser Part Number" "603-AC0603FR-1347RL"
+			(at 118.11 52.07 0)
+			(effects
+				(font
